File: Hardware/SparkFun_Opto_Isolator_Breakout.brd (EAGLE design)
At the start: 15.2 x 12.7 mm, 16 parts, among them Q1 NPN, Q2 NPN, U1 OPTOISOLATOR-2SOIC8

Commit message: Replace ILD213T with updated part
Parts:
- R1, R2: device SparkFun-Resistors:0603-RES -> SparkFun-Resistors:0603
- R3, R4, R5, R6: value 10K -> 10k; device SparkFun-Resistors:0603-RES -> SparkFun-Resistors:0603
- U1: value OPTOISOLATOR-2SOIC8 -> ILD213T-IDL213T; device SparkFun-DiscreteSemi:SO08-2 -> SparkFun-DiscreteSemi:SO08
